Commit message: added lidar and green wheels

File: catkin_ws/src/my_robot/urdf/my_robot.xacro (robot description, xacro)
@@ -56,5 +56,5 @@
   </link>
 <link name='left_wheel'>
-    <pose>0 0 0.1 0 0 0</pose>
+    <pose>0 0 0 0 0 0</pose>
     <inertial>
       <mass value="5.0"/>
@@ -88,5 +88,5 @@
   </joint>
 <link name='right_wheel'>
-    <pose>0 0 0.1 0 0 0</pose>
+    <pose>0 0 0 0 0 0</pose>
     <inertial>
       <mass value="5.0"/>
@@ -120,5 +120,5 @@
   </joint>
 <link name='camera'>
-    <pose>0 0 0.1 0 0 0</pose>
+    <pose>0 0 0 0 0 0</pose>
     <inertial>
       <mass value="5.0"/>
@@ -136,5 +136,5 @@
       </geometry>
     </collision>
-    <visual name='right_wheel_visual'>
+    <visual name='camera_visual'>
       <origin xyz="0 0 0" rpy=" 0 0 0"/>
       <geometry>
@@ -151,3 +151,41 @@
     <dynamics damping="1.0" friction="1.0"/>
   </joint>
+<link name='hokuyo'>
+    <pose>0 0 0 0 0 0</pose>
+    <inertial>
+      <mass value="1e-5"/>
+      <origin xyz="0.0 0 0" rpy="0.0 0 0"/>
+      <inertia
+	ixx="1e-6" ixy="0" ixz="0"
+	iyy="1e-6" iyz="0"
+	izz="1e-6"
+      />
+    </inertial>
+    <collision name='collision'>
+      <origin xyz="0 0 0" rpy=" 0 0 0"/>
+      <geometry>
+        <box size="0.1 0.1 0.1"/>
+      </geometry>
+    </collision>
+    <visual name='hokuyo_visual'>
+      <origin xyz="0 0 0" rpy=" 0 0 0"/>
+      <geometry>
+        <mesh filename="package://my_robot/meshes/hokuyo.dae"/>
+      </geometry>
+    </visual>
+  </link>
+ <joint type="fixed" name="hokuyo_joint">
+    <origin xyz="0.15 0 0.1" rpy="0 0 0"/>
+    <child link="hokuyo"/>
+    <parent link="chassis"/>
+    <axis xyz="0 1 0" rpy="0 0 0"/>
+    <limit effort="10000" velocity="1000"/>
+    <dynamics damping="1.0" friction="1.0"/>
+  </joint>
+<gazebo reference="left_wheel">
+    <material>Gazebo/Green</material>
+</gazebo>
+<gazebo reference="right_wheel">
+    <material>Gazebo/Green</material>
+</gazebo>
 </robot>
